Commit message: update sensor tilting

File: urdf/dpoom.urdf.xacro (robot description, xacro)
@@ -167,4 +167,6 @@
   </link>
   <joint name="camera_rgb_joint" type="fixed">
+    <!--You can tilt the sensor by changing the value of pitch-->
+    <!--Ex) <origin xyz="0.003 0.011 0.009" rpy="0 0.3 0"/>-->
     <origin xyz="0.003 0.011 0.009" rpy="0 0 0"/>
     <parent link="camera_link"/>

Commit message: Update dpoom.urdf.xacro

File: urdf/dpoom.urdf.xacro (robot description, xacro)
@@ -167,6 +167,6 @@
   </link>
   <joint name="camera_rgb_joint" type="fixed">
-    <!--You can tilt the sensor by changing the value of pitch-->
-    <!--Ex) <origin xyz="0.003 0.011 0.009" rpy="0 0.3 0"/>-->
+    <!--You can tilt the sensor by changing the value of pitch
+        Ex) <origin xyz="0.003 0.011 0.009" rpy="0 0.3 0"/>-->
     <origin xyz="0.003 0.011 0.009" rpy="0 0 0"/>
     <parent link="camera_link"/>

Commit message: Add files via upload

File: urdf/dpoom.urdf.xacro (robot description, xacro)
@@ -154,5 +154,11 @@
   </link>
   <joint name="camera_joint" type="fixed">
-    <origin xyz="0.073 -0.011 0.097" rpy="0 0 0"/>
+    <!--You can change the hight of the sensor by changing the value of origin z.
+        Total view-height is sum of this value and "camera_link"'s origin z value, which is 0.013
+        Also, for visualization, the change in this part should be considered in "camera_rgb_frame".
+        (Original height is 0.12m, so z should be 0.12 - 0.013 = 0.107)
+     Ex) <origin xyz="0.073 -0.011 0.107" rpy="0 0 0"/>
+     -->
+    <origin xyz="0.073 -0.011 0.107" rpy="0 0 0"/>
     <parent link="base_link"/>
     <child link="camera_link"/>
@@ -168,5 +174,6 @@
   <joint name="camera_rgb_joint" type="fixed">
     <!--You can tilt the sensor by changing the value of pitch
-        Ex) <origin xyz="0.003 0.011 0.009" rpy="0 0.3 0"/>-->
+    Ex) <origin xyz="0.003 0.011 0.009" rpy="0 0.3 0"/>
+    -->
     <origin xyz="0.003 0.011 0.009" rpy="0 0 0"/>
     <parent link="camera_link"/>
@@ -174,6 +181,13 @@
   </joint>
   <link name="camera_rgb_frame">
-    <visual>
-      <origin xyz="0 0 0" rpy="-1.57 0 -1.57"/>
+    <!--Original value of visual origin is xyz="0 0 -0.01"
+        if you changed the sensor height in "camera_joint", z should be deducted by the
+        height change.
+    EX) if you change the sensor height to 13cm(0.13m), which means that you changed
+        "camera_joint" z from 0.107 to 0.117, the visual z origin should be changed
+        from -0.01 to -0.11
+    -->
+    <visual>
+      <origin xyz="0 0 -0.01" rpy="-1.57 0 -1.57"/>
       <geometry>
         <mesh filename="package://dpoom_gazebo/meshes/sensors/d435.dae" scale="1 1 1"/>
