Commit message: orca and morp for dynamic obs, including goal-stop option

File: urdf/turtlebot3_waffle_pi.gazebo.xacro (robot description, xacro)
@@ -135,5 +135,5 @@
   </gazebo>
 <!--link : https://www.raspberrypi.org/documentation/hardware/camera/-->
-  <gazebo reference="camera_rgb_frame">
+  <!-- <gazebo reference="camera_rgb_frame">
     <sensor name="camera" type="depth">
       <update_rate>20</update_rate>
@@ -153,6 +153,4 @@
         <baseline>0.2</baseline>
         <alwaysOn>true</alwaysOn>
-        <!-- Keep this zero, update_rate in the parent <sensor> tag
-          will control the frame rate. -->
         <updateRate>0.0</updateRate>
         <cameraName>camera_ir</cameraName>
@@ -177,4 +175,4 @@
       </plugin>
     </sensor>
-  </gazebo>
+  </gazebo> -->
 </robot>

File: urdf/turtlebot3_waffle_pi.urdf.xacro (robot description, xacro)
@@ -164,5 +164,5 @@
     </inertial>
   </link>
-  <joint name="camera_joint" type="fixed">
+  <!-- <joint name="camera_joint" type="fixed">
     <origin xyz="0.073 -0.011 0.084" rpy="0 0 0"/>
     <parent link="base_link"/>
@@ -188,4 +188,4 @@
     <child link="camera_rgb_optical_frame"/>
   </joint>
-  <link name="camera_rgb_optical_frame"/>
+  <link name="camera_rgb_optical_frame"/> -->
 </robot>
